File: PICO-blue-chords-pcb/PICO-blue-chords-pcb.kicad_pcb (KiCad board)
At the start: 2 copper layers, 119.4 x 97.8 mm, 27 parts

Commit message: Upgraded to use SDK and added missing PCB tracks.
Connections:
- A1 pad 36: 3V3 -> 3v3PWR
- Brd1 pad 2: 3v3 -> 3v3PWR
- Brd2 pad 2: 3v3 -> 3v3PWR
Routing:
- net 3v3PWR: track 0.00 -> 214.9 mm
- net Control: track 0.00 -> 172.2 mm
- net Thumb: track 0.00 -> 122.5 mm
- net SDA: track 114.9 -> 142.8 mm
- net SCL: track 141.0 -> 158.8 mm
- net Ring: track 69.5 -> 86.7 mm
- net Little: track 143.7 -> 129.8 mm
Other:
- outline, holes or cut-outs redrawn
